File: hardware/baseband-module/lpf-3GHz/KiCad/TG_LPF_3GHz.kicad_sch (KiCad schematic)
At the start: 17 parts, among them J1 IN, J2 OUT

Commit message: Add positions CSV file for control module components in KiCad
Other:
- note added: "Substrate: FR4 0.8mm S1000H-TG155 (JLC-3)"
- note removed: "Substrate: FR4 0.8mm"
Changed lines of the file:
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@@
 		)
 	)
-	(text "Substrate: FR4 0.8mm"
+	(text "Substrate: FR4 0.8mm S1000H-TG155  (JLC-3)"
 		(exclude_from_sim no)
-		(at 189.23 168.91 0)
+		(at 201.93 168.91 0)
 		(effects
 			(font
